File: kicad/valle.sch (KiCad schematic (older format))
At the start: 8 parts, among them IC1 ATMEGA8-P, IC2 L293D, P1 CONN_2

Commit message: схема максимальная
Parts:
- removed C1: CP1, symbol CP1
- removed D1: LED, symbol LED
- added C1: CAPAPOL, symbol CAPAPOL
- added C2, C3, C4: C, symbol C
- added P1, P2: CONN_6, symbol CONN_6
- added P3: CONN_5X2, symbol CONN_5X2
- added R1, R2, R3: R, symbol R
- added U1: LM7905, symbol LM7905
- added UART1: CONN_2, symbol CONN_2
- added X1: CRYSTAL, symbol CRYSTAL
- renumbered P1 to POWER1
Connections:
- net labels added: EN, VD+
- net labels removed: DGND, VCC
- wire segments 79 -> 155
- no-connect marks 18 -> 1
Other:
- moved on the sheet: POWER1

Commit message: схема упрощённая
Parts:
- removed C3, C4: C, symbol C
- removed U1: LM7905, symbol LM7905
- removed X1: CRYSTAL, symbol CRYSTAL
- added XT1: CONN_2, symbol CONN_2
Connections:
- wire segments 155 -> 148
Other:
- moved on the sheet: C1, C2, POWER1
Changed lines of the file:
@@
-EESchema Schematic File Version 2  date Ср. 09 янв. 2013 22:22:30
+EESchema Schematic File Version 2  date Ср. 09 янв. 2013 22:48:33
 LIBS:power
 LIBS:device
@@
 Comment4 ""
 $EndDescr
+Connection ~ 5750 5650
+Wire Wire Line
+	5750 6400 5750 5650
+Wire Wire Line
+	3400 3350 3400 3300
+Wire Wire Line
+	3400 3300 3000 3300
+Wire Wire Line
+	2050 1800 2050 1900
 Wire Wire Line
 	8700 5450 8700 5300
@@
 Wire Wire Line
 	7650 4550 5850 4550
-Connection ~ 5700 5650
-Wire Wire Line
-	5750 6400 5700 6400
-Wire Wire Line
-	5700 6400 5700 5650
 Connection ~ 5950 5350
 Wire Wire Line
@@
 	2800 2850 3400 2850
 Wire Wire Line
-	3400 3150 3400 3050
-Wire Wire Line
-	3400 3050 3000 3050
-Connection ~ 2450 3350
-Wire Wire Line
-	2450 3350 2250 3350
-Wire Wire Line
-	2250 3350 2250 3450
-Wire Wire Line
 	5300 2950 5950 2950
 Wire Wire Line
@@
 Wire Wire Line
 	6200 3350 5300 3350
-Connection ~ 2100 1900
+Connection ~ 2050 1800
 Wire Wire Line
 	4350 5750 4350 5250
 Wire Wire Line
-	1700 1450 1400 1450
-Wire Wire Line
-	1400 1450 1400 1300
-Wire Wire Line
-	2500 1450 3000 1450
-Wire Wire Line
-	1350 2050 1450 2050
-Wire Wire Line
-	1450 2050 1450 2200
+	1350 1200 1350 1350
+Wire Wire Line
+	1300 1950 1400 1950
+Wire Wire Line
+	1400 1950 1400 2100
 Wire Wire Line
 	8350 4850 8350 5300
@@
 	7850 2100 7850 950
 Wire Wire Line
-	1350 1850 1450 1850
-Wire Wire Line
-	2100 2000 2100 1750
-Wire Wire Line
-	1450 1850 1450 1450
-Connection ~ 1450 1450
-Wire Wire Line
-	2650 1500 2650 1450
-Connection ~ 2650 1450
-Wire Wire Line
-	1700 1850 1700 1900
-Wire Wire Line
-	1700 1900 2650 1900
+	1300 1750 1400 1750
+Wire Wire Line
+	1400 1750 1400 1350
+Connection ~ 1400 1350
+Wire Wire Line
+	2600 1400 2600 1350
+Connection ~ 2600 1350
+Wire Wire Line
+	1650 1750 1650 1800
+Wire Wire Line
+	1650 1800 2600 1800
 Wire Wire Line
 	6000 4100 6000 3450
@@
 	4950 1500 4950 1350
 Wire Wire Line
-	2600 3050 2450 3050
-Wire Wire Line
-	2600 3650 2450 3650
-Wire Wire Line
-	2450 3650 2450 3050
-Wire Wire Line
-	3000 3650 3400 3650
-Wire Wire Line
-	3400 3650 3400 3350
-Wire Wire Line
 	3400 2650 2950 2650
 Wire Wire Line
@@
 Wire Wire Line
 	7100 5450 7100 6000
+Wire Wire Line
+	8700 4550 7950 4550
+Wire Wire Line
+	7950 4550 7950 5450
+Wire Wire Line
+	5750 4050 5750 4750
+Wire Wire Line
+	5750 4750 8700 4750
+Wire Wire Line
+	8350 5300 8450 5300
+Wire Wire Line
+	1350 1350 2950 1350
+Connection ~ 1650 1350
+Wire Wire Line
+	3400 3150 3000 3150
+Wire Wire Line
+	3000 3150 3000 3100
+Wire Wire Line
+	5850 5750 5850 6400
 Connection ~ 5850 5750
-Wire Wire Line
-	5850 6400 5850 5750
-Wire Wire Line
-	8700 4550 7950 4550
-Wire Wire Line
-	7950 4550 7950 5450
-Wire Wire Line
-	5750 4050 5750 4750
-Wire Wire Line
-	5750 4750 8700 4750
-Wire Wire Line
-	8350 5300 8450 5300
-$Comp
-L GND #PWR?
+$Comp
+L CONN_2 XT1
+U 1 1 50ED9B2D
+P 2650 3200
+F 0 "XT1" V 2600 3200 40  0000 C CNN
+F 1 "CONN_2" V 2700 3200 40  0000 C CNN
+	1    2650 3200
+	-1   0    0    1
+$EndComp
+Text Label 7850 1100 0    60   ~ 0
+VD+
+$Comp
+L CAPAPOL C1
+U 1 1 50EAA03D
+P 1650 1550
+F 0 "C1" H 1700 1650 50  0000 L CNN
+F 1 "CAPAPOL" H 1700 1450 50  0000 L CNN
+	1    1650 1550
+	1    0    0    -1
+$EndComp
+$Comp
+L GND #PWR01
 U 1 1 50ED7B45
 P 8700 5450
-F 0 "#PWR?" H 8700 5450 30  0001 C CNN
+F 0 "#PWR01" H 8700 5450 30  0001 C CNN
 F 1 "GND" H 8700 5380 30  0001 C CNN
 	1    8700 5450
@@
 $EndComp
 $Comp
-L GND #PWR?
+L GND #PWR02
 U 1 1 50ED79E3
 P 7100 6000
-F 0 "#PWR?" H 7100 6000 30  0001 C CNN
+F 0 "#PWR02" H 7100 6000 30  0001 C CNN
 F 1 "GND" H 7100 5930 30  0001 C CNN
 	1    7100 6000
@@
 $EndComp
 $Comp
-L GND #PWR5
+L GND #PWR03
 U 1 1 50EAAE96
 P 2950 2700
-F 0 "#PWR5" H 2950 2700 30  0001 C CNN
+F 0 "#PWR03" H 2950 2700 30  0001 C CNN
 F 1 "GND" H 2950 2630 30  0001 C CNN
 	1    2950 2700
@@
 Text Label 2950 2850 0    60   ~ 0
 VD+
-$Comp
-L CRYSTAL X1
-U 1 1 50EAADF3
-P 3000 3350
-F 0 "X1" H 3000 3500 60  0000 C CNN
-F 1 "CRYSTAL" H 3000 3200 60  0000 C CNN
-	1    3000 3350
-	0    1    1    0
-$EndComp
-$Comp
-L GND #PWR4
-U 1 1 50EAADD4
-P 2250 3450
-F 0 "#PWR4" H 2250 3450 30  0001 C CNN
-F 1 "GND" H 2250 3380 30  0001 C CNN
-	1    2250 3450
-	1    0    0    -1
-$EndComp
-$Comp
-L C C4
-U 1 1 50EAADBF
-P 2800 3650
-F 0 "C4" H 2850 3750 50  0000 L CNN
-F 1 "C" H 2850 3550 50  0000 L CNN
-	1    2800 3650
-	0    -1   -1   0
-$EndComp
-$Comp
-L C C3
-U 1 1 50EAADB3
-P 2800 3050
-F 0 "C3" H 2850 3150 50  0000 L CNN
-F 1 "C" H 2850 2950 50  0000 L CNN
-	1    2800 3050
-	0    1    1    0
-$EndComp
 $Comp
 L CONN_6 P1
@@
 L C C2
 U 1 1 50EAA07C
-P 2650 1700
-F 0 "C2" H 2700 1800 50  0000 L CNN
-F 1 "C" H 2700 1600 50  0000 L CNN
-	1    2650 1700
-	1    0    0    -1
-$EndComp
-$Comp
-L CAPAPOL C1
-U 1 1 50EAA03D
-P 1700 1650
-F 0 "C1" H 1750 1750 50  0000 L CNN
-F 1 "CAPAPOL" H 1750 1550 50  0000 L CNN
-	1    1700 1650
-	1    0    0    -1
-$EndComp
-$Comp
-L GND #PWR10
+P 2600 1600
+F 0 "C2" H 2650 1700 50  0000 L CNN
+F 1 "C" H 2650 1500 50  0000 L CNN
+	1    2600 1600
+	1    0    0    -1
+$EndComp
+$Comp
+L GND #PWR04
 U 1 1 50E17B17
 P 7950 5450
-F 0 "#PWR10" H 7950 5450 30  0001 C CNN
+F 0 "#PWR04" H 7950 5450 30  0001 C CNN
 F 1 "GND" H 7950 5380 30  0001 C CNN
 	1    7950 5450
@@
 $EndComp
 $Comp
-L GND #PWR6
+L GND #PWR05
 U 1 1 50E17A76
 P 4350 5750
-F 0 "#PWR6" H 4350 5750 30  0001 C CNN
+F 0 "#PWR05" H 4350 5750 30  0001 C CNN
 F 1 "GND" H 4350 5680 30  0001 C CNN
 	1    4350 5750
@@
 VD+
 $Comp
-L +5V #PWR1
+L +5V #PWR06
 U 1 1 50E1680D
-P 1400 1300
-F 0 "#PWR1" H 1400 1390 20  0001 C CNN
-F 1 "+5V" H 1400 1390 30  0000 C CNN
-	1    1400 1300
+P 1350 1200
+F 0 "#PWR06" H 1350 1290 20  0001 C CNN
+F 1 "+5V" H 1350 1290 30  0000 C CNN
+	1    1350 1200
 	1    0    0    -1
 $EndComp
@@
 VD+
 $Comp
-L GND #PWR3
+L GND #PWR07
 U 1 1 50E1666A
-P 2100 2000
-F 0 "#PWR3" H 2100 2000 30  0001 C CNN
-F 1 "GND" H 2100 1930 30  0001 C CNN
-	1    2100 2000
-	1    0    0    -1
-$EndComp
-Text Label 2800 1450 0    60   ~ 0
-VD+
-$Comp
-L LM7905 U1
-U 1 1 50E16631
-P 2100 1500
-F 0 "U1" H 2250 1305 60  0000 C CNN
-F 1 "LM7905" H 2100 1700 60  0000 C CNN
-	1    2100 1500
-	1    0    0    -1
-$EndComp
-$Comp
-L GND #PWR2
+P 2050 1900
+F 0 "#PWR07" H 2050 1900 30  0001 C CNN
+F 1 "GND" H 2050 1830 30  0001 C CNN
+	1    2050 1900
+	1    0    0    -1
+$EndComp
+Text Label 2750 1350 0    60   ~ 0
+VD+
+$Comp
+L GND #PWR08
 U 1 1 50DAE2E9
-P 1450 2200
-F 0 "#PWR2" H 1450 2200 30  0001 C CNN
-F 1 "GND" H 1450 2130 30  0001 C CNN
-	1    1450 2200
+P 1400 2100
+F 0 "#PWR08" H 1400 2100 30  0001 C CNN
+F 1 "GND" H 1400 2030 30  0001 C CNN
+	1    1400 2100
 	1    0    0    -1
 $EndComp
@@
 L CONN_2 POWER1
 U 1 1 50DAE2CD
-P 1000 1950
-F 0 "POWER1" V 950 1950 40  0000 C CNN
-F 1 "CONN_2" V 1050 1950 40  0000 C CNN
-	1    1000 1950
+P 950 1850
+F 0 "POWER1" V 900 1850 40  0000 C CNN
+F 1 "CONN_2" V 1000 1850 40  0000 C CNN
+	1    950  1850
 	-1   0    0    1
 $EndComp
 $Comp
-L +5V #PWR8
-U 1 1 50DADEB7
-P 7850 950
-F 0 "#PWR8" H 7850 1040 20  0001 C CNN
-F 1 "+5V" H 7850 1040 30  0000 C CNN
-	1    7850 950
-	1    0    0    -1
-$EndComp
-$Comp
-L GND #PWR9
+L GND #PWR09
 U 1 1 50DAC666
 P 7950 2950
-F 0 "#PWR9" H 7950 2950 30  0001 C CNN
+F 0 "#PWR09" H 7950 2950 30  0001 C CNN
 F 1 "GND" H 7950 2880 30  0001 C CNN
 	1    7950 2950
@@
 $EndComp
 $Comp
-L GND #PWR7
+L GND #PWR010
 U 1 1 50DAC652
 P 6050 3000
-F 0 "#PWR7" H 6050 3000 30  0001 C CNN
+F 0 "#PWR010" H 6050 3000 30  0001 C CNN
 F 1 "GND" H 6050 2930 30  0001 C CNN
 	1    6050 3000

Commit message: разведённая плата
Parts:
- removed R1: R, symbol R
Connections:
- wire segments 148 -> 146

Commit message: before branch
Connections:
- wire segments 146 -> 158
- no-connect marks 1 -> 2
Changed lines of the file:
@@
-EESchema Schematic File Version 2  date Чт. 10 янв. 2013 14:31:07
+EESchema Schematic File Version 2  date Пт. 11 янв. 2013 10:50:48
 LIBS:power
 LIBS:device
@@
 Sheet 1 1
 Title ""
-Date "10 jan 2013"
+Date "11 jan 2013"
 Rev ""
 Comp ""
@@
 $EndDescr
 Wire Wire Line
+	8700 4750 5750 4750
+Wire Wire Line
+	7650 4650 8700 4650
+Wire Wire Line
 	3400 2450 3400 2250
 Connection ~ 5850 5750
@@
 Connection ~ 1650 1350
 Wire Wire Line
-	2950 1350 1350 1350
+	2950 1350 2600 1350
+Wire Wire Line
+	2600 1350 1650 1350
+Wire Wire Line
+	1650 1350 1400 1350
+Wire Wire Line
+	1400 1350 1350 1350
 Wire Wire Line
 	8450 5300 8350 5300
 Wire Wire Line
-	8700 4750 5750 4750
-Wire Wire Line
 	5750 4750 5750 4050
 Wire Wire Line
@@
 	7100 5450 7100 6000
 Wire Wire Line
-	6300 5650 5300 5650
+	6300 5650 5750 5650
+Wire Wire Line
+	5750 5650 5300 5650
 Wire Wire Line
 	5300 5650 5300 4750
 Wire Wire Line
-	6300 5350 5550 5350
+	6300 5350 5950 5350
+Wire Wire Line
+	5950 5350 5550 5350
 Wire Wire Line
 	5550 5350 5550 4550
@@
 	6000 3450 6000 4100
 Wire Wire Line
-	2600 1800 1650 1800
+	2600 1800 2050 1800
+Wire Wire Line
+	2050 1800 1650 1800
 Wire Wire Line
 	1650 1800 1650 1750
@@
 	6050 3000 6050 2800
 Wire Wire Line
-	4300 1900 4300 2150
+	4300 1900 4300 2050
+Wire Wire Line
+	4300 2050 4300 2150
 Connection ~ 6250 2800
 Wire Wire Line
-	6250 2900 6250 2700
+	6250 2900 6250 2800
+Wire Wire Line
+	6250 2800 6250 2700
 Wire Wire Line
 	6250 2900 6400 2900
@@
 	7750 2800 7950 2800
 Wire Wire Line
-	7750 2900 7750 2700
+	7750 2900 7750 2800
+Wire Wire Line
+	7750 2800 7750 2700
 Wire Wire Line
 	4300 5050 4300 5250
@@
 	1350 1350 1350 1200
 Wire Wire Line
-	4350 5250 4350 5750
+	4350 5250 4350 5550
+Wire Wire Line
+	4350 5550 4350 5750
 Connection ~ 2050 1800
 Wire Wire Line
@@
 	5450 4650 5450 5750
 Wire Wire Line
-	5450 5750 6300 5750
+	5450 5750 5850 5750
+Wire Wire Line
+	5850 5750 6300 5750
 Wire Wire Line
 	5950 6400 5950 5350
@@
 	7650 4550 7650 4650
 Wire Wire Line
-	7650 4650 8700 4650
-Wire Wire Line
-	8450 5450 8450 5200
+	8450 5450 8450 5300
+Wire Wire Line
+	8450 5300 8450 5200
 Wire Wire Line
 	8450 5200 8700 5200
@@
 	5750 6400 5750 5650
 Connection ~ 5750 5650
+NoConn ~ 6300 5450
 $Comp
 L CONN_2 XT1

Commit message: готовая плата
Parts:
- removed XT1: CONN_2, symbol CONN_2
- added C3, C4: C, symbol C
- added P4: CONN_6, symbol CONN_6
- added X1: CRYSTAL, symbol CRYSTAL
Connections:
- wire segments 158 -> 155
